Commit message: fix: correct WebGL→Genesis coordinate transformation in URDF
Update URDF generator and test scripts:
- URDF rpy: "-1.5708 3.14159 0" (X:-90°, Y:180°)
- WebGL(X=left,Y=up,Z=forward) → Genesis(X=right,Y=forward,Z=up)
- Transformation baked into URDF, no euler needed at load time

File: simulator/assets/meshes/parts/stampfly.urdf (robot description, URDF)
Before this commit: robot stampfly, 5 links, 4 joints
Joints:
- joint prop0_joint: origin xyz=0.0325 0.0325 0.01 rpy=0 0 0 -> xyz=0 0 0 rpy=0 0 0
- joint prop1_joint: origin xyz=-0.0325 -0.0325 0.01 rpy=0 0 0 -> xyz=0 0 0 rpy=0 0 0
- joint prop2_joint: origin xyz=-0.0325 0.0325 0.01 rpy=0 0 0 -> xyz=0 0 0 rpy=0 0 0
- joint prop3_joint: origin xyz=0.0325 -0.0325 0.01 rpy=0 0 0 -> xyz=0 0 0 rpy=0 0 0
