Commit message: fix: adjust collision box and increase torque gain
- Lower collision box origin to z=0 and increase height to 35mm
  so bottom is at z=-17.5mm, covering the leg tips
- Increase MAX_TORQUE from 5e-5 to 2e-4 Nm (4x)

File: simulator/assets/meshes/parts/stampfly_fixed.urdf (robot description, URDF)
Before this commit: robot stampfly_fixed, 1 links, 0 joints
Links:
- link base_link: geometry collision box size=0.08 0.08 0.035; visual mesh filename=battery.stl scale=0.001 0.001 0.001

Commit message: fix: set URDF mass to 35g to match documentation

File: simulator/assets/meshes/parts/stampfly_fixed.urdf (robot description, URDF)
Before this commit: robot stampfly_fixed, 1 links, 0 joints
Links:
- link base_link: mass 0.034 -> 0.035
